File: ecoBeat Hardware/PCB_03/_saved_ecoBeat_3.sch (KiCad schematic (older format))
At the start: 24 parts, among them IC1 ATTINY85-P, J1 RJ45, P1 CONN_01X06, P3 CONN_01X02, SW1 SW_PUSH, SW2 SW_PUSH, U1 ESP-12E, U2 AP1117D33

Commit message: PCB_03
Parts:
- removed C2: 100nF, Discret:CP36V, symbol C
- added D?: D, symbol D
- added R10: 10k, Resistors_ThroughHole:Resistor_Horizontal_RM7mm, symbol R
Connections:
- net ESPRST: now also P1.1 (P1)
- net GND: no longer R1.2
- net VCC: now also P3.2 (P2), D?.2 (A), R10.2; no longer C1.1, C4.1, D3.2 (A), IC1.8 (VCC), J1.2, R2.1, R3.1, U1.11 (GPIO2), U1.2 (ADC), U1.3 (CH_PD), U1.8 (VCC), U2.2 (VO)
- net at C3.1, U2.3 (VI): now also D?.1 (K); no longer P3.2 (P2)
- new net: J1.2, R3.1
- new net: R10.1, U1.11 (GPIO2)
- new net 3.3: C1.1, C4.1, D3.2 (A), IC1.8 (VCC), R1.2, R2.1, U1.2 (ADC), U1.3 (CH_PD), U1.8 (VCC), U2.2 (VO)
- no-connect marks 15 -> 14
Other:
- moved on the sheet: P3
