File: ecoBeat Hardware/PCB_03/ecoBeat_3.kicad_pcb (KiCad board)
At the start: 2 copper layers, 120.2 x 129.4 mm, 24 parts, among them IC1 ATTINY85-P, J1 RJ45, P1 CONN_01X06, P3 CONN_01X02, SW1 SW_PUSH, SW2 SW_PUSH, U1 ESP-12E, U2 AP1117D33

Commit message: gerber
Routing:
- net GND: track 58.5 -> 32.1 mm
- removed copper zone on F.Cu, net GND
