File: ecoBeat Hardware/PCB_03/ecoBeat_3.kicad_pcb (KiCad board)
At the start: 2 copper layers, 30.9 x 86 mm, 25 parts, among them IC1 ATTINY85-P, J1 RJ45, P1 CONN_01X06, P3 CONN_01X02, SW1 SW_PUSH, SW2 SW_PUSH, U1 ESP-12E, U2 AP1117D33

Commit message: mandado a fabricar PCBWay
Parts:
- REF**: value MountingHole_2-5mm -> H2mm
- U2: value AP1117D33 -> 1117
Other:
- board text removed: "pulsito"
