File: ecoBeat Hardware/PCB_03/ecoBeat_3.kicad_pcb (KiCad board)
At the start: 2 copper layers, 120.2 x 129.4 mm, 24 parts, among them IC1 ATTINY85-P, J1 RJ45, P1 CONN_01X06, P3 CONN_01X02, SW1 SW_PUSH, SW2 SW_PUSH, U1 ESP-12E, U2 AP1117D33

Commit message: master
Parts:
- U1: footprint ESP8266:ESP-07v2 -> ESP8266:ESP-12E
- moved IC1 0.25 mm to (158.1, 111.8)
Other:
- board size 120.2 x 129.4 mm -> 30.9 x 86 mm

Commit message: master
Parts:
- added REF**: MountingHole_2-5mm, Mounting_Holes:MountingHole_2-5mm, F.Cu at (169.9, 128.1)
Routing:
- net GND: track 32.1 -> 15.6 mm
- added copper zone on F.Cu, net GND
Other:
- outline, holes or cut-outs redrawn
Changed lines of the file:
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@@
 (kicad_pcb (version 4) (host pcbnew 4.0.2+dfsg1-stable)
   (general
-    (links 57)
+    (links 58)
     (no_connects 0)
-    (area 145.109999 57.889999 176.200001 144.040001)
+    (area 144.145 57.15 177.19512 145.415001)
     (thickness 1.6)
-    (drawings 17)
-    (tracks 134)
+    (drawings 16)
+    (tracks 129)
     (zones 0)
-    (modules 24)
+    (modules 25)
     (nets 28)
   )
@@
     (mod_text_size 1 1)
     (mod_text_width 0.15)
-    (pad_size 4 3)
-    (pad_drill 0)
+    (pad_size 3 3)
+    (pad_drill 2.2)
     (pad_to_mask_clearance 0.2)
     (aux_axis_origin 0 0)
@@
     (add_net "Net-(P1-Pad5)")
     (add_net "Net-(R9-Pad1)")
-    (add_net "Net-(U1-Pad17)")
-    (add_net "Net-(U1-Pad18)")
-    (add_net "Net-(U1-Pad19)")
-    (add_net "Net-(U1-Pad20)")
-    (add_net "Net-(U1-Pad21)")
-    (add_net "Net-(U1-Pad22)")
     (add_net "Net-(U1-Pad7)")
     (add_net RSTTINY)
@@
       (effects (font (size 1 1) (thickness 0.15)))
     )
-    (fp_text value ESP-12E (at 6.35 6.35) (layer F.Fab) hide
+    (fp_text value ESP-12E (at 6.985 14.605) (layer F.Fab) hide
       (effects (font (size 1 1) (thickness 0.15)))
     )
@@
       (effects (font (size 1 1) (thickness 0.15)))
     )
-    (fp_text value LED (at 1.3 -2.9 180) (layer F.Fab)
+    (fp_text value LED (at 1.27 1.905 180) (layer F.Fab)
       (effects (font (size 1 1) (thickness 0.15)))
     )
@@
     (fp_arc (start 1.311 0.034) (end 3.051 0.994) (angle 110) (layer F.SilkS) (width 0.15))
     (fp_arc (start 1.301 0.034) (end 2.335 1.094) (angle 87.5) (layer F.SilkS) (width 0.15))
-    (fp_text user K (at -1.69 1.74 180) (layer F.SilkS)
+    (fp_text user K (at 4.445 -1.27 180) (layer F.SilkS)
       (effects (font (size 1 1) (thickness 0.15)))
     )
@@
       (effects (font (size 1 1) (thickness 0.15)))
     )
-    (fp_text value LED (at 1.3 -2.9 180) (layer F.Fab)
+    (fp_text value LED (at 1.27 1.905 180) (layer F.Fab)
       (effects (font (size 1 1) (thickness 0.15)))
     )
@@
     (fp_arc (start 1.311 0.034) (end 3.051 0.994) (angle 110) (layer F.SilkS) (width 0.15))
     (fp_arc (start 1.301 0.034) (end 2.335 1.094) (angle 87.5) (layer F.SilkS) (width 0.15))
-    (fp_text user K (at -1.69 1.74 180) (layer F.SilkS)
+    (fp_text user K (at 4.445 -1.27 180) (layer F.SilkS)
       (effects (font (size 1 1) (thickness 0.15)))
     )
@@
       (effects (font (size 1 1) (thickness 0.15)))
     )
-    (fp_text value LED (at 1.3 -2.9 180) (layer F.Fab)
+    (fp_text value LED (at 1.27 1.905 180) (layer F.Fab)
       (effects (font (size 1 1) (thickness 0.15)))
     )
@@
     (fp_arc (start 1.311 0.034) (end 3.051 0.994) (angle 110) (layer F.SilkS) (width 0.15))
     (fp_arc (start 1.301 0.034) (end 2.335 1.094) (angle 87.5) (layer F.SilkS) (width 0.15))
-    (fp_text user K (at -1.69 1.74 180) (layer F.SilkS)
+    (fp_text user K (at 4.445 -1.27 180) (layer F.SilkS)
       (effects (font (size 1 1) (thickness 0.15)))
     )
@@
     (descr "Resistor, Axial,  RM 7.62mm, 1/3W,")
     (tags "Resistor Axial RM 7.62mm 1/3W R3")
-    (fp_text reference R7 (at 4.05892 -3.50012 270) (layer F.SilkS)
+    (fp_text reference R7 (at 0 2.54 270) (layer F.SilkS)
       (effects (font (size 1 1) (thickness 0.15)))
     )
@@
     )
   )
+  (module Mounting_Holes:MountingHole_2-5mm (layer F.Cu)
+    (at 169.855 128.065)
+    (descr "Mounting hole, Befestigungsbohrung, 2,5mm, No Annular, Kein Restring,")
+    (tags "Mounting hole, Befestigungsbohrung, 2,5mm, No Annular, Kein Restring,")
+    (fp_text reference REF** (at 0 -3.50012) (layer F.SilkS)
+      (effects (font (size 1 1) (thickness 0.15)))
+    )
+    (fp_text value MountingHole_2-5mm (at 0.09906 3.59918) (layer F.Fab)
+      (effects (font (size 1 1) (thickness 0.15)))
+    )
+    (fp_circle (center 0 0) (end 2.5 0) (layer Cmts.User) (width 0.381))
+    (pad 1 thru_hole circle (at 0 0) (size 3 3) (drill 2.2) (layers *.Cu)
+      (net 1 GND))
+  )
   (gr_line (start 176.125 57.965) (end 176.125 68.465) (angle 90) (layer Edge.Cuts) (width 0.15))
   (gr_line (start 176.125 133.44) (end 176.125 143.965) (angle 90) (layer Edge.Cuts) (width 0.15))
@@
   (gr_line (start 146.16 69.465) (end 146.16 132.465) (angle 90) (layer Edge.Cuts) (width 0.15))
   (gr_line (start 175.15 69.465) (end 175.15 132.465) (angle 90) (layer Edge.Cuts) (width 0.15))
-  (gr_circle (center 169.855 128.065) (end 170.955 128.065) (layer Edge.Cuts) (width 0.15))
   (gr_line (start 145.185 143.965) (end 176.125 143.965) (angle 90) (layer Edge.Cuts) (width 0.15))
   (gr_line (start 145.185 57.965) (end 176.125 57.965) (angle 90) (layer Edge.Cuts) (width 0.15))
-  (segment (start 158.369 104.14) (end 160.655 104.14) (width 0.8) (layer F.Cu) (net 1))
-  (segment (start 165.735 113.665) (end 168.275 113.665) (width 0.8) (layer F.Cu) (net 1))
-  (segment (start 164.465 112.395) (end 165.735 113.665) (width 0.8) (layer F.Cu) (net 1))
-  (segment (start 164.465 107.95) (end 164.465 112.395) (width 0.8) (layer F.Cu) (net 1))
-  (segment (start 160.655 104.14) (end 164.465 107.95) (width 0.8) (layer F.Cu) (net 1))
   (segment (start 173.5 138.515) (end 173.5 123.875) (width 0.8) (layer B.Cu) (net 1))
   (segment (start 173.5 123.875) (end 172.815 123.19) (width 0.8) (layer B.Cu) (net 1))
@@
     (polygon
       (pts
-        (xy 177.165 145.415) (xy 144.145 145.415) (xy 144.145 57.15) (xy 177.165 57.15) (xy 177.165 145.415)
+        (xy 177.8 146.05) (xy 143.51 146.05) (xy 143.51 56.515) (xy 177.8 56.515) (xy 177.8 146.05)
       )
     )
+  )
+  (zone (net 1) (net_name GND) (layer F.Cu) (hatch edge 0.508)
+    (connect_pads (clearance 0.508))
+    (min_thickness 0.254)
+    (fill yes (arc_segments 16) (thermal_gap 0.508) (thermal_bridge_width 0.508))
+    (polygon
+      (pts
+        (xy 178.435 146.685) (xy 142.875 146.685) (xy 142.875 55.88) (xy 178.435 55.88) (xy 178.435 146.685)
+      )
+    )
+  )
+  (zone (net 0) (net_name "") (layer F.Cu) (hatch full 0.508)
+    (connect_pads (clearance 0.508))
+    (min_thickness 0.254)
+    (keepout (tracks not_allowed) (vias not_allowed) (copperpour not_allowed))
+    (fill (arc_segments 16) (thermal_gap 0.508) (thermal_bridge_width 0.508))
+    (polygon
+      (pts
+        (xy 175.895 65.405) (xy 145.415 65.405) (xy 145.415 58.42) (xy 175.895 58.42) (xy 175.895 65.405)
+      )
+    )

Commit message: 1117 volteado
Parts:
- U2: moved to F.Cu
- turned U2 to 0 degrees
Routing:
- net VCC: track 141.3 -> 135.9 mm
- net Net-(C3-Pad1): track 14.3 -> 10.1 mm
Other:
- board text added: "EndeF ecoBeat 1"
- board text added: "pulsito"

Commit message: attiny Firmware_3_actualizacion
Parts:
- removed C4: 10uF, Capacitors_ThroughHole:C_Radial_D5_L11_P2
- removed D2, D3: LED, LEDs:LED-3MM
- removed D4: D, Diodes_ThroughHole:Diode_DO-35_SOD27_Horizontal_RM10
- removed REF**: MountingHole_2-5mm, Mounting_Holes:MountingHole_2-5mm
- added C2: 10uF, Capacitors_ThroughHole:C_Radial_D5_L6_P2.5, F.Cu at (171.6, 116.3)
- added P2: CONN_01X02, Connect:bornier2, F.Cu at (171.1, 140.1)
- added R10: 220, Resistors_SMD:R_0805, F.Cu at (123.6, 104.6)
- added R11: 10k, Resistors_SMD:R_0805, F.Cu at (172.8, 80.9)
- C3: footprint Capacitors_ThroughHole:C_Radial_D5_L11_P2 -> Capacitors_ThroughHole:C_Radial_D5_L6_P2.5
- D1: value LED -> D; footprint LEDs:LED-3MM -> Diodes_ThroughHole:Diode_DO-35_SOD27_Horizontal_RM10
- IC1: footprint Housings_DIP:DIP-8_W7.62mm -> Housings_DIP:DIP-8_W7.62mm_LongPads
- P3: value CONN_01X02 -> CONN_01X04; footprint Connect:bornier2 -> Pin_Headers:Pin_Header_Straight_1x04
- R1, R2, R8: footprint Resistors_ThroughHole:Resistor_Horizontal_RM7mm -> Resistors_SMD:R_0805
- R3: value 10k -> 6.8k; footprint Resistors_ThroughHole:Resistor_Horizontal_RM7mm -> Resistors_SMD:R_0805
- R4: value 6.8k -> 12k; footprint Resistors_ThroughHole:Resistor_Horizontal_RM7mm -> Resistors_SMD:R_0805
- R5: value 12k -> 10k; footprint Resistors_ThroughHole:Resistor_Horizontal_RM7mm -> Resistors_SMD:R_0805
- R6, R7: value 220 -> 10k; footprint Resistors_ThroughHole:Resistor_Horizontal_RM7mm -> Resistors_SMD:R_0805
- R9: value 10k -> 220; footprint Resistors_ThroughHole:Resistor_Horizontal_RM7mm -> Resistors_SMD:R_0805
- SW1, SW2: footprint Buttons_Switches_ThroughHole:SW_PUSH_SMALL -> switch:SW_PUSH_SMALL
- U1: value ESP-12E -> ESP-12F
- moved SW1 85.5 mm to (223.0, 152.9), turned to 0 degrees
- moved SW2 83.5 mm to (228.1, 117.5), turned to 0 degrees
- moved R1 73.5 mm to (225.0, 147.3), turned to 0 degrees
- moved R8 71.9 mm to (101.0, 107.2), turned to 0 degrees
- moved R7 71.4 mm to (220.9, 147.3), turned to 0 degrees
- moved R5 66.4 mm to (119.3, 114.9), turned to 180 degrees
- moved P3 59.9 mm to (119.9, 107.2)
- moved R4 58.0 mm to (119.9, 111.3), turned to 270 degrees
- moved R2 56.6 mm to (103.9, 113.7), turned to 270 degrees
- moved R3 54.3 mm to (172.7, 69.7), turned to 180 degrees
- moved R6 53.0 mm to (221.2, 115.6)
- moved C1 49.2 mm to (181.0, 155.1), turned to 0 degrees
- moved IC1 43.7 mm to (114.6, 114.8)
- moved R9 43.3 mm to (123.6, 102.1), turned to 0 degrees
- moved D1 21.2 mm to (182.6, 122.0), turned to 270 degrees
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Connections:
- C1 pad 1: VCC -> 3.3
- C3 pad 1: Net-(C3-Pad1) -> 3.3
- D1 pad 1: Net-(D1-Pad1) -> VCC
- D1 pad 2: L1 -> Net-(D1-Pad2)
- IC1 pad 2: RX1 -> RXD
- IC1 pad 3: TX1 -> TXD
- IC1 pad 8: VCC -> 3.3
- J1 pad 1: Net-(J1-Pad1) -> (no net)
- J1 pad 2: VCC -> 3.3
- J1 pad 3: Net-(J1-Pad3) -> (no net)
- J1 pad 4: Net-(J1-Pad4) -> (no net)
- J1 pad 7: Net-(J1-Pad7) -> (no net)
- J1 pad 8: Net-(J1-Pad8) -> (no net)
- P1 pad 4: Net-(P1-Pad4) -> (no net)
- P1 pad 5: Net-(P1-Pad5) -> 3.3
- R1 pad 1: Net-(IC1-Pad7) -> 3.3
- R1 pad 2: GND -> ESPRST
- R2 pad 1: VCC -> Net-(IC1-Pad7)
- R2 pad 2: ESPRST -> 3.3
- R3 pad 1: VCC -> Net-(P1-Pad3)
- R3 pad 2: RSTTINY -> RXD
- R4 pad 1: Net-(P1-Pad3) -> GND
- R5 pad 1: GND -> 3.3
- R5 pad 2: RXD -> RSTTINY
- R6 pad 1: GND -> Net-(R6-Pad1)
- R6 pad 2: Net-(D1-Pad1) -> VCC
- R7 pad 1: GND -> Net-(R7-Pad1)
- R7 pad 2: Net-(D2-Pad1) -> 3.3
- R8 pad 1: GND -> Net-(P3-Pad4)
- R8 pad 2: Net-(D3-Pad1) -> L1
- R9 pad 1: Net-(R9-Pad1) -> Net-(P3-Pad3)
- R9 pad 2: VCC -> L2
- SW1 pad 1: Net-(R9-Pad1) -> ESPRST
- SW2 pad 1: ESPRST -> Net-(R6-Pad1)
- U1 pad 10: GND -> Net-(R11-Pad1)
- U1 pad 11: VCC -> (no net)
- U1 pad 12: Net-(R9-Pad1) -> Net-(R6-Pad1)
- U1 pad 13: RX1 -> (no net)
- U1 pad 14: TX1 -> (no net)
- U1 pad 2: VCC -> 3.3
- U1 pad 3: VCC -> Net-(R7-Pad1)
- U1 pad 7: Net-(U1-Pad7) -> (no net)
- U1 pad 8: VCC -> 3.3
- U2 pad 2: VCC -> 3.3
- U2 pad 3: Net-(C3-Pad1) -> VCC
Routing:
- net VCC: track 135.9 -> 0.00 mm
- net ESPRST: track 72.7 -> 0.00 mm
- net RSTTINY: track 48.7 -> 0.00 mm
- net RX1: track 41.2 -> 0.00 mm
- net TX1: track 40.6 -> 0.00 mm
- net L2: track 37.9 -> 0.00 mm
- net INT1: track 35.2 -> 0.00 mm
- net TXD: track 27.1 -> 0.00 mm
- net Net-(R9-Pad1): track 22.5 -> 0.00 mm
- net L1: track 22.2 -> 0.00 mm
- net Net-(IC1-Pad7): track 20.3 -> 0.00 mm
- net GND: track 15.6 -> 0.00 mm
- net RXD: track 15.3 -> 0.00 mm
- net Net-(D1-Pad1): track 13.1 -> 0.00 mm
- net Net-(C3-Pad1): track 10.1 -> 0.00 mm
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Other:
- board text removed: "pulsito"
