File: ecoBeat Hardware/PCB_03/ecoBeat_3.sch (KiCad schematic (older format))
At the start: 24 parts, among them IC1 ATTINY85-P, J1 RJ45, P1 CONN_01X06, P3 CONN_01X02, SW1 SW_PUSH, SW2 SW_PUSH, U1 ESP-12E, U2 AP1117D33

Commit message: PCB_03
Parts:
- removed D4: D, Diodes_ThroughHole:Diode_DO-35_SOD27_Horizontal_RM10, symbol D
- added R10: 10k, Resistors_ThroughHole:Resistor_Horizontal_RM7mm, symbol R
Connections:
- net GND: no longer R1.2
- net VCC: now also C3.1, P3.2 (P2), U2.3 (VI), R10.2; no longer C1.1, C4.1, D3.2 (A), IC1.8 (VCC), J1.2, R2.1, R3.1, U1.11 (GPIO2), U1.2 (ADC), U1.3 (CH_PD), U1.8 (VCC), U2.2 (VO)
- new net: J1.2, R3.1
- new net: R10.1, U1.11 (GPIO2)
- new net 3.3: C1.1, C4.1, D3.2 (A), IC1.8 (VCC), R1.2, R2.1, U1.2 (ADC), U1.3 (CH_PD), U1.8 (VCC), U2.2 (VO)
- no-connect marks 15 -> 14
Changed lines of the file:
@@
 L GND #PWR05
 U 1 1 5A843508
-P 4800 2550
-F 0 "#PWR05" H 4800 2300 50  0001 C CNN
-F 1 "GND" H 4800 2400 50  0000 C CNN
-F 2 "" H 4800 2550 50  0000 C CNN
-F 3 "" H 4800 2550 50  0000 C CNN
-	1    4800 2550
-	1    0    0    -1
-$EndComp
-$Comp
-L VCC #PWR06
-U 1 1 5A843537
-P 2050 1150
-F 0 "#PWR06" H 2050 1000 50  0001 C CNN
-F 1 "VCC" H 2050 1300 50  0000 C CNN
-F 2 "" H 2050 1150 50  0000 C CNN
-F 3 "" H 2050 1150 50  0000 C CNN
-	1    2050 1150
-	1    0    0    -1
-$EndComp
-$Comp
-L GND #PWR07
+P 5150 2550
+F 0 "#PWR05" H 5150 2300 50  0001 C CNN
+F 1 "GND" H 5150 2400 50  0000 C CNN
+F 2 "" H 5150 2550 50  0000 C CNN
+F 3 "" H 5150 2550 50  0000 C CNN
+	1    5150 2550
+	1    0    0    -1
+$EndComp
+$Comp
+L GND #PWR06
 U 1 1 5A843719
 P 2050 2800
-F 0 "#PWR07" H 2050 2550 50  0001 C CNN
+F 0 "#PWR06" H 2050 2550 50  0001 C CNN
 F 1 "GND" H 2050 2650 50  0000 C CNN
 F 2 "" H 2050 2800 50  0000 C CNN
@@
 $EndComp
 $Comp
-L VCC #PWR08
+L VCC #PWR07
 U 1 1 5A8449B1
 P 5500 2050
-F 0 "#PWR08" H 5500 1900 50  0001 C CNN
+F 0 "#PWR07" H 5500 1900 50  0001 C CNN
 F 1 "VCC" H 5500 2200 50  0000 C CNN
 F 2 "" H 5500 2050 50  0000 C CNN
@@
 RXD
 $Comp
-L GND #PWR09
+L GND #PWR08
 U 1 1 5A84637A
 P 3950 4650
-F 0 "#PWR09" H 3950 4400 50  0001 C CNN
+F 0 "#PWR08" H 3950 4400 50  0001 C CNN
 F 1 "GND" H 3950 4500 50  0000 C CNN
 F 2 "" H 3950 4650 50  0000 C CNN
@@
 	4700 2050 5100 2050
 Wire Wire Line
-	4700 2150 5450 2150
-Wire Wire Line
-	4700 2250 4800 2250
-Wire Wire Line
-	4700 2350 4800 2350
+	4700 2350 5150 2350
 Wire Wire Line
 	9200 1150 9200 1250
@@
 Wire Wire Line
 	3050 6100 2800 6100
-Wire Wire Line
-	1800 6000 3050 6000
 Wire Wire Line
 	1800 5950 1800 6550
@@
 L1
 $Comp
-L VCC #PWR010
-U 1 1 5A84809C
-P 3150 6700
-F 0 "#PWR010" H 3150 6550 50  0001 C CNN
-F 1 "VCC" H 3150 6850 50  0000 C CNN
-F 2 "" H 3150 6700 50  0000 C CNN
-F 3 "" H 3150 6700 50  0000 C CNN
-	1    3150 6700
-	1    0    0    -1
-$EndComp
-$Comp
-L GND #PWR011
+L GND #PWR09
 U 1 1 5A8480D0
 P 1900 6300
-F 0 "#PWR011" H 1900 6050 50  0001 C CNN
+F 0 "#PWR09" H 1900 6050 50  0001 C CNN
 F 1 "GND" H 1900 6150 50  0000 C CNN
 F 2 "" H 1900 6300 50  0000 C CNN
@@
 Wire Wire Line
 	5900 5800 5750 5800
-Wire Wire Line
-	5900 5250 5900 5800
-$Comp
-L GND #PWR012
+$Comp
+L GND #PWR010
 U 1 1 5A848325
 P 5900 6450
-F 0 "#PWR012" H 5900 6200 50  0001 C CNN
+F 0 "#PWR010" H 5900 6200 50  0001 C CNN
 F 1 "GND" H 5900 6300 50  0000 C CNN
 F 2 "" H 5900 6450 50  0000 C CNN
 F 3 "" H 5900 6450 50  0000 C CNN
 	1    5900 6450
-	1    0    0    -1
-$EndComp
-$Comp
-L VCC #PWR013
-U 1 1 5A848359
-P 5900 5250
-F 0 "#PWR013" H 5900 5100 50  0001 C CNN
-F 1 "VCC" H 5900 5400 50  0000 C CNN
-F 2 "" H 5900 5250 50  0000 C CNN
-F 3 "" H 5900 5250 50  0000 C CNN
-	1    5900 5250
 	1    0    0    -1
 $EndComp
@@
 Connection ~ 9350 3750
 Connection ~ 8550 3750
-$Comp
-L VCC #PWR014
-U 1 1 5A84A447
-P 9450 3650
-F 0 "#PWR014" H 9450 3500 50  0001 C CNN
-F 1 "VCC" H 9450 3800 50  0000 C CNN
-F 2 "" H 9450 3650 50  0000 C CNN
-F 3 "" H 9450 3650 50  0000 C CNN
-	1    9450 3650
-	1    0    0    -1
-$EndComp
 Wire Wire Line
 	8550 4150 8550 4200
@@
 Connection ~ 8950 4200
 $Comp
-L GND #PWR015
+L GND #PWR011
 U 1 1 5A84A948
 P 8950 4300
-F 0 "#PWR015" H 8950 4050 50  0001 C CNN
+F 0 "#PWR011" H 8950 4050 50  0001 C CNN
 F 1 "GND" H 8950 4150 50  0000 C CNN
 F 2 "" H 8950 4300 50  0000 C CNN
@@
 Connection ~ 8600 5500
 $Comp
-L GND #PWR016
+L GND #PWR012
 U 1 1 5A84C7C1
 P 8600 6000
-F 0 "#PWR016" H 8600 5750 50  0001 C CNN
+F 0 "#PWR012" H 8600 5750 50  0001 C CNN
 F 1 "GND" H 8600 5850 50  0000 C CNN
 F 2 "" H 8600 6000 50  0000 C CNN
@@
 Wire Wire Line
 	10150 5500 10150 5350
-$Comp
-L VCC #PWR017
-U 1 1 5A84CF1B
-P 10150 5350
-F 0 "#PWR017" H 10150 5200 50  0001 C CNN
-F 1 "VCC" H 10150 5500 50  0000 C CNN
-F 2 "" H 10150 5350 50  0000 C CNN
-F 3 "" H 10150 5350 50  0000 C CNN
-	1    10150 5350
-	1    0    0    -1
-$EndComp
 Wire Wire Line
 	3150 6800 3150 6700
 NoConn ~ 2850 2250
-NoConn ~ 8850 1400
 NoConn ~ 1600 6550
 NoConn ~ 1700 6550
@@
 	1300 7350 1300 7450
 $Comp
-L GND #PWR018
+L GND #PWR013
 U 1 1 5A8537A8
 P 1300 7450
-F 0 "#PWR018" H 1300 7200 50  0001 C CNN
+F 0 "#PWR013" H 1300 7200 50  0001 C CNN
 F 1 "GND" H 1300 7300 50  0000 C CNN
 F 2 "" H 1300 7450 50  0000 C CNN
@@
 NoConn ~ 4000 4350
 Wire Wire Line
-	4800 2250 4800 2550
-Connection ~ 4800 2350
+	5150 2250 5150 2550
+Connection ~ 5150 2350
 $Comp
 L CONN_01X02 P3
@@
 	-1   0    0    1
 $EndComp
-Connection ~ 2450 6000
-Connection ~ 5900 5450
 Wire Wire Line
 	8200 3950 8200 3750
 Wire Wire Line
-	8000 3950 8200 3950
+	7600 3950 8200 3950
 Wire Wire Line
 	7600 4050 8200 4050
@@
 	8200 4050 8200 4200
 Connection ~ 8550 4200
-$Comp
-L GND #PWR019
-U 1 1 5AA7B386
-P 1800 5600
-F 0 "#PWR019" H 1800 5350 50  0001 C CNN
-F 1 "GND" H 1800 5450 50  0000 C CNN
-F 2 "" H 1800 5600 50  0000 C CNN
-F 3 "" H 1800 5600 50  0000 C CNN
-	1    1800 5600
-	-1   0    0    1
-$EndComp
 $Comp
 L SW_PUSH SW1
@@
 	5800 1850 5800 2150
 $Comp
-L GND #PWR020
+L GND #PWR014
 U 1 1 5AA7C0A8
 P 5800 2150
-F 0 "#PWR020" H 5800 1900 50  0001 C CNN
+F 0 "#PWR014" H 5800 1900 50  0001 C CNN
 F 1 "GND" H 5800 2000 50  0000 C CNN
 F 2 "" H 5800 2150 50  0000 C CNN
@@
 	1    0    0    -1
 $EndComp
-$Comp
-L D D4
-U 1 1 5AA8E873
-P 7850 3950
-F 0 "D4" H 7850 4050 50  0000 C CNN
-F 1 "D" H 7850 3850 50  0000 C CNN
-F 2 "Diodes_ThroughHole:Diode_DO-35_SOD27_Horizontal_RM10" H 7850 3950 50  0001 C CNN
-F 3 "" H 7850 3950 50  0000 C CNN
-	1    7850 3950
-	-1   0    0    1
-$EndComp
-Wire Wire Line
-	7700 3950 7600 3950
+Wire Wire Line
+	3050 6000 1800 6000
+Wire Wire Line
+	5900 5800 5900 5250
+$Comp
+L R R10
+U 1 1 5AA94F3E
+P 5250 2150
+F 0 "R10" V 5330 2150 50  0000 C CNN
+F 1 "10k" V 5250 2150 50  0000 C CNN
+F 2 "Resistors_ThroughHole:Resistor_Horizontal_RM7mm" V 5180 2150 50  0001 C CNN
+F 3 "" H 5250 2150 50  0000 C CNN
+	1    5250 2150
+	0    -1   -1   0
+$EndComp
+Wire Wire Line
+	5450 2150 5400 2150
+Wire Wire Line
+	4700 2150 5100 2150
+Text GLabel 9450 3650 1    60   Input ~ 0
+3.3
+Text GLabel 10150 5350 1    60   Input ~ 0
+3.3
+Text GLabel 5900 5250 1    60   Input ~ 0
+3.3
+Text GLabel 1800 5600 1    60   Input ~ 0
+3.3
+Text GLabel 2050 1150 1    60   Input ~ 0
+3.3
+$Comp
+L VCC #PWR015
+U 1 1 5AA98C74
+P 7700 3550
+F 0 "#PWR015" H 7700 3400 50  0001 C CNN
+F 1 "VCC" H 7700 3700 50  0000 C CNN
+F 2 "" H 7700 3550 50  0000 C CNN
+F 3 "" H 7700 3550 50  0000 C CNN
+	1    7700 3550
+	1    0    0    -1
+$EndComp
+Wire Wire Line
+	7700 3550 7700 3950
+Connection ~ 7700 3950
+Wire Wire Line
+	4700 2250 5150 2250
 $EndSCHEMATC

Commit message: gerber
Parts:
- added D?: D, symbol D
Connections:
- net VCC: now also D?.2 (A); no longer C3.1, U2.3 (VI)
- new net: C3.1, D?.1 (K), U2.3 (VI)
Changed lines of the file:
@@
 	8200 3950 8200 3750
 Wire Wire Line
-	7600 3950 8200 3950
+	7600 3950 7800 3950
 Wire Wire Line
 	7600 4050 8200 4050
@@
 $EndComp
 Wire Wire Line
-	7700 3550 7700 3950
+	7700 3950 7700 3550
 Connection ~ 7700 3950
 Wire Wire Line
 	4700 2250 5150 2250
+$Comp
+L D D?
+U 1 1 5AAA6483
+P 7950 3950
+F 0 "D?" H 7950 4050 50  0000 C CNN
+F 1 "D" H 7950 3850 50  0000 C CNN
+F 2 "" H 7950 3950 50  0000 C CNN
+F 3 "" H 7950 3950 50  0000 C CNN
+	1    7950 3950
+	-1   0    0    1
+$EndComp
+Wire Wire Line
+	8200 3950 8100 3950
 $EndSCHEMATC
