File: ecoBeat Hardware/PCB_03/ecoBeat_3.sch (KiCad schematic (older format))
At the start: 25 parts, among them IC1 ATTINY85-P, J1 RJ45, P1 CONN_01X06, P3 CONN_01X02, SW1 SW_PUSH, SW2 SW_PUSH, U1 ESP-12E, U2 AP1117D33

Commit message: master
Parts:
- removed U1: ESP-12E, ESP8266:ESP-12E, symbol ESP-12E
- added U1: ESP-12F, ESP8266:ESP-12E, symbol ESP-12F
- D1: renamed from D?; footprint (none) -> Diodes_ThroughHole:Diode_DO-35_SOD27_Horizontal_RM10
- IC1: footprint Housings_DIP:DIP-8_W7.62mm -> Housings_DIP:DIP-8_W7.62mm_LongPads
- SW1: renamed from SW2; footprint Buttons_Switches_ThroughHole:SW_PUSH_SMALL -> switch:SW_PUSH_SMALL
- SW2: renamed from SW1; footprint Buttons_Switches_ThroughHole:SW_PUSH_SMALL -> switch:SW_PUSH_SMALL
- renumbered C3 to C2, C4 to C3, D1 to D2, D2 to D3, D3 to D4, P3 to P2, R2 to R1, R8 to R10, R1 to R2, R4 to R3, R5 to R4, R3 to R5, R9 to R6, R10 to R7, R6 to R8, R7 to R9
Other:
- moved on the sheet: J1, R2, R5

Commit message: mandado a fabricar PCBWay
Parts:
- D2, D3, D4: symbol LED -> LED-RESCUE-ecoBeat_3
Changed lines of the file:
@@
 EESchema Schematic File Version 2
+LIBS:ecoBeat_3-rescue
 LIBS:power
 LIBS:device
@@
 $EndComp
 $Comp
-L LED D2
+L LED-RESCUE-ecoBeat_3 D2
 U 1 1 5A83FD4B
 P 9350 4900
@@
 $EndComp
 $Comp
-L LED D3
+L LED-RESCUE-ecoBeat_3 D3
 U 1 1 5A83FEA4
 P 9350 5200
@@
 $EndComp
 $Comp
-L LED D4
+L LED-RESCUE-ecoBeat_3 D4
 U 1 1 5A83FF0F
 P 9350 5500
