File: ecoBeat Hardware/PCB_03/ecoBeat_3.sch (KiCad schematic (older format))
At the start: 25 parts, among them IC1 ATTINY85-P, J1 RJ45, P1 CONN_01X06, P2 CONN_01X02, SW1 SW_PUSH, SW2 SW_PUSH, U1 ESP-12F, U2 AP1117D33

Commit message: attiny Firmware_3_actualizacion
Parts:
- removed D2, D3, D4: LED, LEDs:LED-3MM, symbol LED
- added P3: CONN_01X04, Pin_Headers:Pin_Header_Straight_1x04, symbol CONN_01X04
- added R11: 10k, Resistors_SMD:R_0805, symbol R
- C1: footprint Discret:CP36V -> Capacitors_ThroughHole:C_Disc_D3_P2.5
- C2, C3: footprint Capacitors_ThroughHole:C_Disc_D3_P2.5 -> Capacitors_ThroughHole:C_Radial_D5_L6_P2.5
- R1, R10, R2, R3, R4, R5, R6, R7, R8, R9: footprint Resistors_ThroughHole:Resistor_Horizontal_RM7mm -> Resistors_SMD:R_0805
Connections:
- net 3.3: now also P1.5 (P5), R10.2, R7.2; no longer U1.3 (CH_PD)
- net GND: now also P3.1 (P1), R11.2; no longer R10.1, R8.1, R9.1, U1.10 (GPIO15)
- net L1: now also R8.2
- net L2: now also R9.2
- net RXD: now also IC1.2 (PB3(XTAL1/CLKI/OC1B/ADC3/PCINT3))
- net TXD: now also IC1.3 (PB4(XTAL2/CLKO/OC1B/ADC2/PCINT4))
- net VCC: now also C2.1, D1.1 (K), U2.3 (VI); no longer D1.2 (A), P2.2 (P2), R7.2
- net at U1.11 (GPIO2): no longer R7.1
- net RX1: no longer names the net of U1.13 (GPIO4)
- net RX1: no longer IC1.2 (PB3(XTAL1/CLKI/OC1B/ADC3/PCINT3))
- net TX1: no longer names the net of U1.14 (GPIO5)
- net TX1: no longer IC1.3 (PB4(XTAL2/CLKO/OC1B/ADC2/PCINT4))
- new net: P3.2 (P2), R10.1
- new net: P3.3 (P3), R9.1
- new net: P3.4 (P4), R8.1
- new net: D1.2 (A), P2.2 (P2)
- new net: R11.1, U1.10 (GPIO15)
- new net: R7.1, U1.3 (CH_PD)
- no-connect marks 14 -> 16
Other:
- moved on the sheet: R10, R8, R9
